File: AR19_ACME/PCB/ACME_V4.1.brd (EAGLE design)
At the start: 47 x 34.1 mm, 23 parts, among them IC1 Optocoupler DIP, Q1 NGD8201ANT4G, Q2 NGD8201ANT4G

Commit message: ACME V4.2
Routing:
- net 5V: track 7.01 -> 8.51 mm
Other:
- board text added: "Pull up or pull down N-Mosfet - GND P-Mosfet - 12V"
- board text removed: "N-Mosfet - ■ GND P-Mosfet - ■ 12V ■ Pull up or pull down"
Changed lines of the file:
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@@
 <text x="31.05" y="3.75" size="1.778" layer="25" align="center">10</text>
 <text x="17.25" y="3.75" size="1.778" layer="25" align="center">3</text>
-<text x="36" y="2" size="1.778" layer="22" rot="MR0">N-Mosfet - ■ GND
-P-Mosfet - ■ 12V
-■ Pull up or pull down</text>
+<text x="36" y="-1" size="1.778" layer="22" rot="MR0">Pull up or pull down
+N-Mosfet - GND
+P-Mosfet - 12V
+</text>
 </plain>
 <attributes>
@@
 <contactref element="U$1" pad="5V1_P"/>
 <contactref element="U$5" pad="7"/>
-<wire x1="41" y1="7" x2="41" y2="4.5" width="1" layer="1"/>
-<wire x1="41" y1="4.5" x2="40" y2="3.5" width="1" layer="1"/>
-<wire x1="40" y1="3.5" x2="38.69" y2="3.5" width="1" layer="1"/>
-<wire x1="42.26" y1="8.26" x2="41" y2="7" width="1" layer="1"/>
 <polygon width="0.5" layer="1" pour="cutout">
 <vertex x="38" y="-2"/>
@@
 <vertex x="7.85" y="-2"/>
 </polygon>
+<wire x1="41.35" y1="4.16" x2="40.69" y2="3.5" width="1" layer="1"/>
+<wire x1="38.69" y1="3.5" x2="40.69" y2="3.5" width="1" layer="1"/>
+<wire x1="43.5" y1="8.26" x2="42.5" y2="8.26" width="1" layer="1"/>
+<wire x1="42.5" y1="8.26" x2="41.35" y2="7.11" width="1" layer="1"/>
+<wire x1="41.35" y1="7.11" x2="41.35" y2="4.16" width="1" layer="1"/>
 </signal>
 <signal name="PWM0">
