File: AR19_ACME/PCB/ACME_V4.2.brd (EAGLE design)
At the start: 47 x 34 mm, 23 parts, among them IC1 Optocoupler DIP, Q1 NGD8201ANT4G, Q2 NGD8201ANT4G

Commit message: ACME Ordered
Parts:
- added C1, C2, C3, C4: TACL105K006XTA, 0603_Tantalum_Capacitor:CAPPC1709X100N
- moved N_FET0 0.90 mm to (16.6, 22.6)
- moved P_FET10 0.60 mm to (16.6, 20.6)
- moved N_FET1 0.30 mm to (16.6, 18.8)
Connections:
- net 12V: now also C1.1, C2.1, C3.1, C4.1
- net GND: now also C1.2, C2.2, C3.2, C4.2
Routing:
- net GND: track 24.9 -> 28.2 mm
- net 12V: track 63.4 -> 62.4 mm
